File: drive-signal.kicad_pcb (KiCad board)
At the start: 2 copper layers, 46 x 82.3 mm, 32 parts, among them J1 Conn_01x03_Pin, J10 Conn_01x04_Pin, J11 Conn_01x04_Pin, J12 IMU, J13 I2C2 P1, J14 I2C2 P2, J2 Conn_01x03_Pin, J3 Conn_01x03_Pin, J4 Conn_01x03_Pin, J5 JETSON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

Commit message: vias and cleanup
Parts:
- J7: value Conn_01x02_Pin -> POWER
Routing:
- net I2C2_J_SDA: track 71.0 -> 72.5 mm, vias 2 -> 1
- net I2C2_J_SCL: vias 1 -> 0
- net GND: vias 5 -> 17
Other:
- board text added: "ECCENTRIC ORANGE"

Commit message: done
Parts:
- C1: moved to B.Cu
- moved C1 0.25 mm to (63.8, 72.1)
Routing:
- net +5V: track 175.0 -> 162.4 mm, vias 0 -> 1
- net PWM_RF: track 20.4 -> 15.8 mm
- net I2C1_I_SCL: track 54.0 -> 50.9 mm, vias 2 -> 1
- net PWM_LF: track 32.0 -> 29.6 mm
- net I2C2_J_SDA: track 72.5 -> 70.3 mm
- net PWM_RB: track 29.8 -> 28.7 mm
- net I2C1_I_SDA: track 51.2 -> 52.1 mm, vias 1 -> 0
- net GND: vias 17 -> 3
