File: drive-signal.kicad_sch (KiCad schematic)
At the start: 32 parts, among them J1 Conn_01x03_Pin, J10 Conn_01x04_Pin, J11 Conn_01x04_Pin, J12 IMU, J13 I2C2 P1, J14 I2C2 P2, J2 Conn_01x03_Pin, J3 Conn_01x03_Pin, J4 Conn_01x03_Pin, J5 JETSON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

Commit message: done
Other:
- moved on the sheet: H1, H2, H3, H4
Changed lines of the file:
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@@
   (junction (at 26.67 172.72) (diameter 0) (color 0 0 0 0)
   )
-  (junction (at -17.78 142.24) (diameter 0) (color 0 0 0 0)
+  (junction (at 170.18 148.59) (diameter 0) (color 0 0 0 0)
   )
   (junction (at 185.42 60.96) (diameter 0) (color 0 0 0 0)
@@
   (junction (at 185.42 38.1) (diameter 0) (color 0 0 0 0)
   )
-  (junction (at -17.78 149.86) (diameter 0) (color 0 0 0 0)
+  (junction (at 170.18 156.21) (diameter 0) (color 0 0 0 0)
   )
   (junction (at 26.67 166.37) (diameter 0) (color 0 0 0 0)
@@
   (junction (at 26.67 160.02) (diameter 0) (color 0 0 0 0)
   )
-  (junction (at -17.78 134.62) (diameter 0) (color 0 0 0 0)
+  (junction (at 170.18 140.97) (diameter 0) (color 0 0 0 0)
   )
   (no_connect (at 107.95 63.5))
@@
     (stroke (width 0) (type default))
   )
-  (wire (pts (xy -17.78 134.62) (xy -22.86 134.62))
+  (wire (pts (xy 170.18 140.97) (xy 165.1 140.97))
     (stroke (width 0) (type default))
   )
@@
     (stroke (width 0) (type default))
   )
-  (wire (pts (xy -17.78 149.86) (xy -22.86 149.86))
+  (wire (pts (xy 170.18 156.21) (xy 165.1 156.21))
     (stroke (width 0) (type default))
   )
@@
     (stroke (width 0) (type default))
   )
-  (wire (pts (xy -17.78 127) (xy -17.78 134.62))
+  (wire (pts (xy 170.18 133.35) (xy 170.18 140.97))
     (stroke (width 0) (type default))
   )
@@
     (stroke (width 0) (type default))
   )
-  (wire (pts (xy -17.78 134.62) (xy -17.78 142.24))
+  (wire (pts (xy 170.18 140.97) (xy 170.18 148.59))
     (stroke (width 0) (type default))
   )
@@
     (stroke (width 0) (type default))
   )
-  (wire (pts (xy -17.78 149.86) (xy -17.78 156.21))
+  (wire (pts (xy 170.18 156.21) (xy 170.18 162.56))
     (stroke (width 0) (type default))
   )
@@
     (stroke (width 0) (type default))
   )
-  (wire (pts (xy -17.78 127) (xy -22.86 127))
+  (wire (pts (xy 170.18 133.35) (xy 165.1 133.35))
     (stroke (width 0) (type default))
   )
@@
     (stroke (width 0) (type default))
   )
-  (wire (pts (xy -17.78 142.24) (xy -17.78 149.86))
+  (wire (pts (xy 170.18 148.59) (xy 170.18 156.21))
     (stroke (width 0) (type default))
   )
@@
     (stroke (width 0) (type default))
   )
-  (wire (pts (xy -17.78 142.24) (xy -22.86 142.24))
+  (wire (pts (xy 170.18 148.59) (xy 165.1 148.59))
     (stroke (width 0) (type default))
   )
@@
     )
   )
-  (symbol (lib_id "Mechanical:MountingHole_Pad") (at -25.4 134.62 90) (unit 1)
+  (symbol (lib_id "Mechanical:MountingHole_Pad") (at 162.56 140.97 90) (unit 1)
     (in_bom yes) (on_board yes) (dnp no)
-    (property "Reference" "H2" (at -39.37 132.08 90)
-      (effects (font (size 1.27 1.27)))
-    )
-    (property "Value" "MountingHole_Pad" (at -39.37 134.62 90)
-      (effects (font (size 1.27 1.27)))
-    )
-    (property "Footprint" "MountingHole:MountingHole_3.2mm_M3_Pad_Via" (at -25.4 134.62 0)
-      (effects (font (size 1.27 1.27)) hide)
-    )
-    (property "Datasheet" "~" (at -25.4 134.62 0)
+    (property "Reference" "H2" (at 148.59 138.43 90)
+      (effects (font (size 1.27 1.27)))
+    )
+    (property "Value" "MountingHole_Pad" (at 148.59 140.97 90)
+      (effects (font (size 1.27 1.27)))
+    )
+    (property "Footprint" "MountingHole:MountingHole_3.2mm_M3_Pad_Via" (at 162.56 140.97 0)
+      (effects (font (size 1.27 1.27)) hide)
+    )
+    (property "Datasheet" "~" (at 162.56 140.97 0)
       (effects (font (size 1.27 1.27)) hide)
     )
@@
     )
   )
-  (symbol (lib_id "Mechanical:MountingHole_Pad") (at -25.4 142.24 90) (unit 1)
+  (symbol (lib_id "Mechanical:MountingHole_Pad") (at 162.56 148.59 90) (unit 1)
     (in_bom yes) (on_board yes) (dnp no)
-    (property "Reference" "H3" (at -39.37 139.7 90)
-      (effects (font (size 1.27 1.27)))
-    )
-    (property "Value" "MountingHole_Pad" (at -39.37 142.24 90)
-      (effects (font (size 1.27 1.27)))
-    )
-    (property "Footprint" "MountingHole:MountingHole_3.2mm_M3_Pad_Via" (at -25.4 142.24 0)
-      (effects (font (size 1.27 1.27)) hide)
-    )
-    (property "Datasheet" "~" (at -25.4 142.24 0)
+    (property "Reference" "H3" (at 148.59 146.05 90)
+      (effects (font (size 1.27 1.27)))
+    )
+    (property "Value" "MountingHole_Pad" (at 148.59 148.59 90)
+      (effects (font (size 1.27 1.27)))
+    )
+    (property "Footprint" "MountingHole:MountingHole_3.2mm_M3_Pad_Via" (at 162.56 148.59 0)
+      (effects (font (size 1.27 1.27)) hide)
+    )
+    (property "Datasheet" "~" (at 162.56 148.59 0)
       (effects (font (size 1.27 1.27)) hide)
     )
@@
     )
   )
-  (symbol (lib_id "Mechanical:MountingHole_Pad") (at -25.4 127 90) (unit 1)
+  (symbol (lib_id "Mechanical:MountingHole_Pad") (at 162.56 133.35 90) (unit 1)
     (in_bom yes) (on_board yes) (dnp no)
-    (property "Reference" "H1" (at -39.37 124.46 90)
-      (effects (font (size 1.27 1.27)))
-    )
-    (property "Value" "MountingHole_Pad" (at -39.37 127 90)
-      (effects (font (size 1.27 1.27)))
-    )
-    (property "Footprint" "MountingHole:MountingHole_3.2mm_M3_Pad_Via" (at -25.4 127 0)
-      (effects (font (size 1.27 1.27)) hide)
-    )
-    (property "Datasheet" "~" (at -25.4 127 0)
+    (property "Reference" "H1" (at 148.59 130.81 90)
+      (effects (font (size 1.27 1.27)))
+    )
+    (property "Value" "MountingHole_Pad" (at 148.59 133.35 90)
+      (effects (font (size 1.27 1.27)))
+    )
+    (property "Footprint" "MountingHole:MountingHole_3.2mm_M3_Pad_Via" (at 162.56 133.35 0)
+      (effects (font (size 1.27 1.27)) hide)
+    )
+    (property "Datasheet" "~" (at 162.56 133.35 0)
       (effects (font (size 1.27 1.27)) hide)
     )
@@
     )
   )
-  (symbol (lib_id "Mechanical:MountingHole_Pad") (at -25.4 149.86 90) (unit 1)
+  (symbol (lib_id "Mechanical:MountingHole_Pad") (at 162.56 156.21 90) (unit 1)
     (in_bom yes) (on_board yes) (dnp no)
-    (property "Reference" "H4" (at -39.37 147.32 90)
-      (effects (font (size 1.27 1.27)))
-    )
-    (property "Value" "MountingHole_Pad" (at -39.37 149.86 90)
-      (effects (font (size 1.27 1.27)))
-    )
-    (property "Footprint" "MountingHole:MountingHole_3.2mm_M3_Pad_Via" (at -25.4 149.86 0)
-      (effects (font (size 1.27 1.27)) hide)
-    )
-    (property "Datasheet" "~" (at -25.4 149.86 0)
+    (property "Reference" "H4" (at 148.59 153.67 90)
+      (effects (font (size 1.27 1.27)))
+    )
+    (property "Value" "MountingHole_Pad" (at 148.59 156.21 90)
+      (effects (font (size 1.27 1.27)))
+    )
+    (property "Footprint" "MountingHole:MountingHole_3.2mm_M3_Pad_Via" (at 162.56 156.21 0)
+      (effects (font (size 1.27 1.27)) hide)
+    )
+    (property "Datasheet" "~" (at 162.56 156.21 0)
       (effects (font (size 1.27 1.27)) hide)
     )
@@
     )
   )
-  (symbol (lib_id "power:GND") (at -17.78 156.21 0) (unit 1)
-    (in_bom yes) (on_board yes) (dnp no) (fields_autoplaced)
-    (property "Reference" "#PWR026" (at -17.78 162.56 0)
-      (effects (font (size 1.27 1.27)) hide)
-    )
-    (property "Value" "GND" (at -17.78 161.29 0)
-      (effects (font (size 1.27 1.27)))
-    )
-    (property "Footprint" "" (at -17.78 156.21 0)
-      (effects (font (size 1.27 1.27)) hide)
-    )
-    (property "Datasheet" "" (at -17.78 156.21 0)
-      (effects (font (size 1.27 1.27)) hide)
-    )
+  (symbol (lib_id "power:GND") (at 170.18 162.56 0) (unit 1)
+    (in_bom yes) (on_board yes) (dnp no) (fields_autoplaced)
+    (property "Reference" "#PWR026" (at 170.18 168.91 0)
+      (effects (font (size 1.27 1.27)) hide)
+    )
+    (property "Value" "GND" (at 170.18 167.64 0)
+      (effects (font (size 1.27 1.27)))
+    )
+    (property "Footprint" "" (at 170.18 162.56 0)
+      (effects (font (size 1.27 1.27)) hide)
+    )
+    (property "Datasheet" "" (at 170.18 162.56 0)
+      (effects (font (size 1.27 1.27)) hide)
+    )
